Commit message: modified:   README.md 	new file:   config/main.rviz 	new file:   config/my_controllers.yaml 	new file:   description/camera.xacro 	modified:   description/colours.xacro 	new file:   description/lidar.xacro 	modified:   description/robot.urdf.xacro 	new file:   description/ros2_control.xacro 	modified:   launch/launch_sim.launch.py 	modified:   launch/rsp.launch.py 	new file:   worlds/basic.world

File: description/colours.xacro (robot description, xacro)
@@ -12,4 +12,7 @@
     <material name="black">
         <color rgba="0 0 0 1"/>
-</material>
+    </material>
+    <material name="red">
+        <color rgba="1 0 0 1"/>
+    </material>
 </robot>

File: description/robot.urdf.xacro (robot description, xacro)
@@ -1,7 +1,13 @@
 <?xml version="1.0"?>
 <robot xmlns:xacro="http://www.ros.org/wiki/xacro"  name="robot">
+    <xacro:arg name="use_ros2_control" default="true"/>
     <xacro:include filename="inertia_macros.xacro" />
-    <xacro:include filename="gazebo_control.xacro" />
+    <!-- <xacro:include filename="gazebo_control.xacro" /> -->
+    <xacro:if value="$(arg use_ros2_control)">
+        <xacro:include filename="ros2_control.xacro" />
+    </xacro:if>
     <xacro:include filename="robot_core.xacro" />
     <xacro:include filename="colours.xacro" />
+    <xacro:include filename="lidar.xacro" />
+    <xacro:include filename="camera.xacro" />
 </robot>
